File: project/haptic-console-control-unit.kicad_sch (KiCad schematic)
At the start: 30 parts, among them J1 JST-XH-5, J2 JST-XH-5, U1 Teensy 4.1

Commit message: fix erc
Parts:
- renumbered NP to NP1
Connections:
- no-connect marks 19 -> 13
