File: project/haptic-console-control-unit.kicad_sch (KiCad schematic)
At the start: 30 parts, among them J1 JST-XH-5, J2 JST-XH-5, U1 Teensy 4.1

Commit message: more readable
Connections:
- net +3V3: now also S1.2 (Pin_2), S2.2 (Pin_2), S3.2 (Pin_2), S4.2 (Pin_2), S5.2 (Pin_2), S6.2 (Pin_2); no longer S1.5 (Pin_5), S2.5 (Pin_5), S3.5 (Pin_5), S4.5 (Pin_5), S5.5 (Pin_5), S6.5 (Pin_5)
- net +5V: now also S1.3 (Pin_3), S2.3 (Pin_3), S3.3 (Pin_3), S4.3 (Pin_3), S5.3 (Pin_3), S6.3 (Pin_3); no longer S1.4 (Pin_4), S2.4 (Pin_4), S3.4 (Pin_4), S4.4 (Pin_4), S5.4 (Pin_4), S6.4 (Pin_4)
- net GND: now also S1.1 (Pin_1), S2.1 (Pin_1), S3.1 (Pin_1), S4.1 (Pin_1), S5.1 (Pin_1), S6.1 (Pin_1); no longer S1.6 (Pin_6), S2.6 (Pin_6), S3.6 (Pin_6), S4.6 (Pin_6), S5.6 (Pin_6), S6.6 (Pin_6)
- net IRQ1: now also S1.6 (Pin_6); no longer S1.1 (Pin_1)
- net IRQ2: now also S2.6 (Pin_6); no longer S2.1 (Pin_1)
- net IRQ3: now also S3.6 (Pin_6); no longer S3.1 (Pin_1)
- net IRQ4: now also S4.6 (Pin_6); no longer S4.1 (Pin_1)
- net IRQ5: now also S5.6 (Pin_6); no longer S5.1 (Pin_1)
- net IRQ6: now also S6.6 (Pin_6); no longer S6.1 (Pin_1)
- net SCL: now also S1.5 (Pin_5), S2.5 (Pin_5), S3.5 (Pin_5), S4.5 (Pin_5), S5.5 (Pin_5), S6.5 (Pin_5); no longer S1.2 (Pin_2), S2.2 (Pin_2), S3.2 (Pin_2), S4.2 (Pin_2), S5.2 (Pin_2), S6.2 (Pin_2)
- net SDA: now also S1.4 (Pin_4), S2.4 (Pin_4), S3.4 (Pin_4), S4.4 (Pin_4), S5.4 (Pin_4), S6.4 (Pin_4); no longer S1.3 (Pin_3), S2.3 (Pin_3), S3.3 (Pin_3), S4.3 (Pin_3), S5.3 (Pin_3), S6.3 (Pin_3)
