File: project/haptic-console-control-unit.kicad_sch (KiCad schematic)
At the start: 30 parts, among them J1 JST-XH-5, J2 JST-XH-5, U1 Teensy 4.1

Commit message: Add TP1-TP5 test points (SDA/SCL/GND/+3V3/+5V) to schematic and both boards
Schematic: 5 TestPoint symbols wired near the R12/R13 pullup network.
Manufactured board: 5 THT test pads routed around the existing autorouted
copper. Perfboard: real male 2.54mm header pins (not flat pads) at the
board's last column, with S1-S6 shifted one column left to clear them.
Wiring guide and README updated to match; full session notes in CLAUDE.md.

Co-Authored-By: Claude Sonnet 5 <noreply@anthropic.com>
Parts:
- added TP1: TP_SDA, TestPoint:TestPoint_THTPad_D1.5mm_Drill0.7mm, symbol Connector:TestPoint
- added TP2: TP_SCL, TestPoint:TestPoint_THTPad_D1.5mm_Drill0.7mm, symbol Connector:TestPoint
- added TP3: TP_GND, TestPoint:TestPoint_THTPad_D1.5mm_Drill0.7mm, symbol Connector:TestPoint
- added TP4: TP_3V3, TestPoint:TestPoint_THTPad_D1.5mm_Drill0.7mm, symbol Connector:TestPoint
- added TP5: TP_5V, TestPoint:TestPoint_THTPad_D1.5mm_Drill0.7mm, symbol Connector:TestPoint
Connections:
- net +3V3: now also TP4.1
- net +5V: now also TP5.1
- net GND: now also TP3.1
- net SCL: now also TP2.1
- net SDA: now also TP1.1

Commit message: Remap every GPIO to its nearest Teensy pin, fix stale CB4/D13 doc note
Every connector signal (B1-B8, CB1-5, J1/J2, NP1, LED1-5) now sits on
whichever Teensy pin is physically closest to it on the board instead
of a contiguous functional block, solved as a bipartite matching over
Manhattan wire distance. Schematic labels, the manufactured board's
nets/routing, and the perfboard's hand-wiring layout were all
regenerated from the new scripts/pin_map.json; docs and renders follow.

Also drops the panel wiring guide's leftover "CB4 sits on pin 13"
hazard callout, which the remap made false (D13 moved to NP1's row-0
output) - the equivalent warning already lives in the NP1 section.

Co-Authored-By: Claude Sonnet 5 <noreply@anthropic.com>
Connections:
- net D0: now also B1.2 (Pin_2); no longer J1.1 (Pin_1)
- net D1: now also CB1.1 (Pin_1); no longer J1.2 (Pin_2)
- net D10: now also R2.2; no longer CB1.1 (Pin_1)
- net D11: now also CB3.1 (Pin_1); no longer CB2.1 (Pin_1)
- net D12: now also R3.2; no longer CB3.1 (Pin_1)
- net D13: now also NP1.5 (Pin_5); no longer CB4.1 (Pin_1)
- net D2: now also J1.1 (Pin_1); no longer J1.3 (Pin_3)
- net D20: now also B3.2 (Pin_2); no longer B1.2 (Pin_2)
- net D24: now also J2.3 (Pin_3); no longer B5.2 (Pin_2)
- net D25: now also J2.4 (Pin_4); no longer B6.2 (Pin_2)
- net D26: now also CB4.1 (Pin_1); no longer B7.2 (Pin_2)
- net D27: now also NP1.1 (Pin_1); no longer B8.2 (Pin_2)
- net D28: now also R4.2; no longer NP1.1 (Pin_1)
- net D3: now also J1.2 (Pin_2); no longer J1.4 (Pin_4)
- net D31: now also CB5.1 (Pin_1); no longer NP1.4 (Pin_4)
- net D32: now also R5.2; no longer NP1.5 (Pin_5)
- net D34: now also B5.2 (Pin_2); no longer NP1.7 (Pin_7)
- net D35: now also B6.2 (Pin_2); no longer NP1.8 (Pin_8)
- net D36: now also NP1.4 (Pin_4); no longer R3.2
- net D37: now also NP1.6 (Pin_6); no longer R4.2
- net D4: now also J1.3 (Pin_3); no longer J2.1 (Pin_1)
- net D5: now also J1.4 (Pin_4); no longer J2.2 (Pin_2)
- net D6: now also CB2.1 (Pin_1); no longer J2.3 (Pin_3)
- net D7: now also R1.2; no longer J2.4 (Pin_4)
- net D8: now also J2.1 (Pin_1); no longer R1.2
- net D9: now also J2.2 (Pin_2); no longer R2.2
- net IRQ1: now also U1.44 (22_A8_CTX1); no longer U1.37 (15_A1_RX3_SPDIF_IN)
- net IRQ2: now also U1.45 (23_A9_CRX1_MCLK1); no longer U1.38 (16_A2_RX4_SCL1)
- net IRQ4: now also U1.36 (14_A0_TX3_SPDIF_OUT); no longer U1.31 (39_MISO1_OUT1A)
- net IRQ5: now also U1.30 (38_CS1_IN1); no longer U1.32 (40_A16)
- net IRQ6: now also U1.25 (33_MCLK2); no longer U1.33 (41_A17)
- removed net D14: CB5.1 (Pin_1), U1.36 (14_A0_TX3_SPDIF_OUT)
- removed net D22: B3.2 (Pin_2), U1.44 (22_A8_CTX1)
- net D23 renamed D16
- net D16: now also U1.38 (16_A2_RX4_SCL1); no longer U1.45 (23_A9_CRX1_MCLK1)
- removed net D33: NP1.6 (Pin_6), U1.25 (33_MCLK2)
- removed net D38: R5.2, U1.30 (38_CS1_IN1)
- new net D15: B8.2 (Pin_2), U1.37 (15_A1_RX3_SPDIF_IN)
- new net D39: B7.2 (Pin_2), U1.31 (39_MISO1_OUT1A)
- new net D40: NP1.7 (Pin_7), U1.32 (40_A16)
- new net D41: NP1.8 (Pin_8), U1.33 (41_A17)

Commit message: Resync every KiCad artifact to the current pin map (LED4 frozen on D13)
R4's LED jumper was re-landed from R29 (D16 = J1 pin 4, already soldered) to
O29 (D13), clearing the hardware conflict flagged last session. LED4 joins the
frozen set, which now holds 18 already-soldered conductors: B1-B8, J1/J2, LED4,
LED5. Freezing it costs nothing -- the solver had already chosen D13 -- so the
map stays at 1356.3 mm total Manhattan run, 61.0 mm longest wire.

- Schematic: 44 net labels renamed to their GPIO names (D<n>) via delete +
  re-add at identical coordinates. 2244 lines, 141 labels, ERC 0/0, 63 nets,
  all 40 signals verified on their intended U1 pin from the netlist libparts.
- Manufactured board: re-netted from a fresh netlist dump and re-routed via
  DSN -> Freerouting -> SES. 654 segments, 35 vias, DRC 0 violations /
  0 unconnected pads. Needed -mp 40; -mp 6 exited clean at 991.13 with one
  net still unrouted.
- Perfboard: R1-R5 moved upright beside their own CB in KiCad (they had only
  been patched into board_model.json before), 223 back-side jumper legs across
  6 tiers, 0 emit violations, 0 same-tier conflicts. Pristine DRC baseline is
  now 451 (was 478) -- moving the resistors off row 48 removed 27 violations --
  and the wired board's violation multiset is identical to it.
- Gerbers re-exported and re-zipped; all six renders regenerated, with zero
  wire overflow in all six colours confirmed by pixel measurement.
- Docs: wiring-guide.html regenerated (107 connections, 3006 mm, 157 pads /
  223 wires), panel-wiring-guide.html and README.md updated to match.

Co-Authored-By: Claude Opus 5 <noreply@anthropic.com>
Connections:
- net D1: now also B2.2 (Pin_2); no longer CB1.1 (Pin_1)
- net D10: now also NP1.4 (Pin_4); no longer R2.2
- net D11: now also NP1.8 (Pin_8); no longer CB3.1 (Pin_1)
- net D12: now also S4.6 (Pin_6); no longer R3.2
- net D13: now also R4.2; no longer NP1.5 (Pin_5)
- net D15: now also R3.2; no longer B8.2 (Pin_2)
- net D16: now also J1.4 (Pin_4); no longer B4.2 (Pin_2)
- net D2: now also S1.6 (Pin_6); no longer J1.1 (Pin_1)
- net D20: now also J1.3 (Pin_3); no longer B3.2 (Pin_2)
- net D21: now also J1.2 (Pin_2); no longer B2.2 (Pin_2)
- net D24: now also NP1.7 (Pin_7); no longer J2.3 (Pin_3)
- net D25: now also NP1.6 (Pin_6); no longer J2.4 (Pin_4)
- net D26: now also B7.2 (Pin_2); no longer CB4.1 (Pin_1)
- net D27: now also S5.6 (Pin_6); no longer NP1.1 (Pin_1)
- net D28: now also NP1.5 (Pin_5); no longer R4.2
- net D29: now also R5.2; no longer NP1.2 (Pin_2)
- net D3: now also S2.6 (Pin_6); no longer J1.2 (Pin_2)
- net D30: now also B6.2 (Pin_2); no longer NP1.3 (Pin_3)
- net D31: now also S6.6 (Pin_6); no longer CB5.1 (Pin_1)
- net D32: now also B5.2 (Pin_2); no longer R5.2
- net D34: now also CB5.1 (Pin_1); no longer B5.2 (Pin_2)
- net D35: now also NP1.2 (Pin_2); no longer B6.2 (Pin_2)
- net D36: now also NP1.3 (Pin_3); no longer NP1.4 (Pin_4)
- net D37: now also J2.1 (Pin_1); no longer NP1.6 (Pin_6)
- net D39: now also J2.2 (Pin_2); no longer B7.2 (Pin_2)
- net D4: now also B3.2 (Pin_2); no longer J1.3 (Pin_3)
- net D40: now also J2.3 (Pin_3); no longer NP1.7 (Pin_7)
- net D41: now also J2.4 (Pin_4); no longer NP1.8 (Pin_8)
- net D5: now also R1.2; no longer J1.4 (Pin_4)
- net D7: now also S3.6 (Pin_6); no longer R1.2
- net D8: now also B4.2 (Pin_2); no longer J2.1 (Pin_1)
- net D9: now also B8.2 (Pin_2); no longer J2.2 (Pin_2)
- net IRQ1 renamed D22
- net D22: now also J1.1 (Pin_1); no longer S1.6 (Pin_6)
- net IRQ2 renamed D23
- net D23: now also CB1.1 (Pin_1); no longer S2.6 (Pin_6)
- net IRQ3 renamed D17
- net D17: now also R2.2; no longer S3.6 (Pin_6)
- net IRQ4 renamed D14
- net D14: now also CB3.1 (Pin_1); no longer S4.6 (Pin_6)
- net IRQ5 renamed D38
- net D38: now also CB4.1 (Pin_1); no longer S5.6 (Pin_6)
- net IRQ6 renamed D33
- net D33: now also NP1.1 (Pin_1); no longer S6.6 (Pin_6)
Changed lines of the file:
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@@
     (stroke (width 0) (type default))
   )
-  (label "D30" (at 101.6 71.12 0) (effects (font (size 1.27 1.27))))
   (label "LED_ARM" (at 93.98 101.6 0) (effects (font (size 1.27 1.27))))
   (label "SCL" (at 220.98 130.81 0) (effects (font (size 1.27 1.27))))
@@
   (label "D7" (at 24.13 87.63 0) (effects (font (size 1.27 1.27))))
   (label "D35" (at 85.09 120.65 0) (effects (font (size 1.27 1.27))))
-  (label "IRQ3" (at 85.09 90.17 0) (effects (font (size 1.27 1.27))))
   (label "+3V3" (at 24.13 102.87 0) (effects (font (size 1.27 1.27))))
   (label "D21" (at 85.09 80.01 0) (effects (font (size 1.27 1.27))))
-  (label "IRQ6" (at 220.98 158.75 0) (effects (font (size 1.27 1.27))))
   (label "+5V" (at 24.13 137.16 0) (effects (font (size 1.27 1.27))))
   (label "D11" (at 24.13 97.79 0) (effects (font (size 1.27 1.27))))
@@
   (label "D31" (at 24.13 123.19 0) (effects (font (size 1.27 1.27))))
   (label "+5V" (at 220.98 49.53 0) (effects (font (size 1.27 1.27))))
-  (label "IRQ5" (at 220.98 133.35 0) (effects (font (size 1.27 1.27))))
   (label "LED_EN" (at 118.11 101.6 0) (effects (font (size 1.27 1.27))))
   (label "SDA" (at 220.98 128.27 0) (effects (font (size 1.27 1.27))))
@@
   (label "+3V3" (at 220.98 97.79 0) (effects (font (size 1.27 1.27))))
   (label "SDA" (at 85.09 87.63 0) (effects (font (size 1.27 1.27))))
-  (label "D29" (at 101.6 68.58 0) (effects (font (size 1.27 1.27))))
-  (label "D21" (at 107.95 185.42 0) (effects (font (size 1.27 1.27))))
   (label "GND" (at 82.55 134.62 0) (effects (font (size 1.27 1.27))))
   (label "D28" (at 24.13 115.57 0) (effects (font (size 1.27 1.27))))
   (label "GND" (at 220.98 95.25 0) (effects (font (size 1.27 1.27))))
   (label "D6" (at 24.13 85.09 0) (effects (font (size 1.27 1.27))))
-  (label "IRQ3" (at 220.98 82.55 0) (effects (font (size 1.27 1.27))))
   (label "D32" (at 24.13 125.73 0) (effects (font (size 1.27 1.27))))
   (label "+5V" (at 220.98 24.13 0) (effects (font (size 1.27 1.27))))
@@
   (label "D20" (at 85.09 82.55 0) (effects (font (size 1.27 1.27))))
   (label "D12" (at 24.13 100.33 0) (effects (font (size 1.27 1.27))))
-  (label "IRQ2" (at 220.98 57.15 0) (effects (font (size 1.27 1.27))))
   (label "D37" (at 85.09 115.57 0) (effects (font (size 1.27 1.27))))
-  (label "IRQ1" (at 220.98 31.75 0) (effects (font (size 1.27 1.27))))
   (label "D1" (at 24.13 72.39 0) (effects (font (size 1.27 1.27))))
   (label "+3V3" (at 220.98 46.99 0) (effects (font (size 1.27 1.27))))
@@
   (label "D4" (at 24.13 80.01 0) (effects (font (size 1.27 1.27))))
   (label "D5" (at 24.13 82.55 0) (effects (font (size 1.27 1.27))))
-  (label "IRQ4" (at 220.98 107.95 0) (effects (font (size 1.27 1.27))))
   (label "D26" (at 24.13 110.49 0) (effects (font (size 1.27 1.27))))
   (label "GND" (at 24.13 67.31 0) (effects (font (size 1.27 1.27))))
@@
   (label "+3V3" (at 269.24 125.73 180) (effects (font (size 1.27 1.27))))
   (label "+5V" (at 269.24 140.97 180) (effects (font (size 1.27 1.27))))
-  (label "D31" (at 194.31 96.52 0) (effects (font (size 1.27 1.27))))
-  (label "D9" (at 133.35 137.16 0) (effects (font (size 1.27 1.27))))
   (label "D16" (at 85.09 92.71 0) (effects (font (size 1.27 1.27))))
-  (label "IRQ1" (at 85.09 77.47 0) (effects (font (size 1.27 1.27))))
   (label "D41" (at 85.09 105.41 0) (effects (font (size 1.27 1.27))))
-  (label "D40" (at 101.6 81.28 0) (effects (font (size 1.27 1.27))))
-  (label "D25" (at 133.35 142.24 0) (effects (font (size 1.27 1.27))))
-  (label "D34" (at 83.82 167.64 0) (effects (font (size 1.27 1.27))))
-  (label "IRQ2" (at 85.09 74.93 0) (effects (font (size 1.27 1.27))))
-  (label "D12" (at 154.94 123.19 0) (effects (font (size 1.27 1.27))))
-  (label "D35" (at 107.95 167.64 0) (effects (font (size 1.27 1.27))))
-  (label "IRQ5" (at 85.09 113.03 0) (effects (font (size 1.27 1.27))))
-  (label "D8" (at 133.35 134.62 0) (effects (font (size 1.27 1.27))))
-  (label "D7" (at 105.41 123.19 0) (effects (font (size 1.27 1.27))))
-  (label "D15" (at 148.59 167.64 0) (effects (font (size 1.27 1.27))))
-  (label "D3" (at 99.06 137.16 0) (effects (font (size 1.27 1.27))))
-  (label "IRQ6" (at 85.09 125.73 0) (effects (font (size 1.27 1.27))))
   (label "D6" (at 120.65 96.52 0) (effects (font (size 1.27 1.27))))
   (label "D0" (at 83.82 185.42 0) (effects (font (size 1.27 1.27))))
-  (label "D11" (at 146.05 96.52 0) (effects (font (size 1.27 1.27))))
-  (label "D16" (at 148.59 185.42 0) (effects (font (size 1.27 1.27))))
   (label "D15" (at 85.09 95.25 0) (effects (font (size 1.27 1.27))))
-  (label "D10" (at 129.54 123.19 0) (effects (font (size 1.27 1.27))))
-  (label "D32" (at 204.47 123.19 0) (effects (font (size 1.27 1.27))))
-  (label "D2" (at 99.06 134.62 0) (effects (font (size 1.27 1.27))))
-  (label "D37" (at 101.6 78.74 0) (effects (font (size 1.27 1.27))))
-  (label "D1" (at 96.52 96.52 0) (effects (font (size 1.27 1.27))))
-  (label "D13" (at 101.6 76.2 0) (effects (font (size 1.27 1.27))))
-  (label "D27" (at 101.6 66.04 0) (effects (font (size 1.27 1.27))))
-  (label "D5" (at 99.06 142.24 0) (effects (font (size 1.27 1.27))))
-  (label "D24" (at 133.35 139.7 0) (effects (font (size 1.27 1.27))))
-  (label "D36" (at 101.6 73.66 0) (effects (font (size 1.27 1.27))))
-  (label "D41" (at 101.6 83.82 0) (effects (font (size 1.27 1.27))))
   (label "D40" (at 85.09 107.95 0) (effects (font (size 1.27 1.27))))
-  (label "D4" (at 99.06 139.7 0) (effects (font (size 1.27 1.27))))
-  (label "D39" (at 129.54 167.64 0) (effects (font (size 1.27 1.27))))
   (label "D39" (at 85.09 110.49 0) (effects (font (size 1.27 1.27))))
-  (label "D28" (at 180.34 123.19 0) (effects (font (size 1.27 1.27))))
-  (label "D26" (at 171.45 96.52 0) (effects (font (size 1.27 1.27))))
-  (label "IRQ4" (at 85.09 97.79 0) (effects (font (size 1.27 1.27))))
-  (label "D20" (at 129.54 185.42 0) (effects (font (size 1.27 1.27))))
+  (label "D22" (at 85.09 77.47 0) (effects (font (size 1.27 1.27))))
+  (label "D23" (at 85.09 74.93 0) (effects (font (size 1.27 1.27))))
+  (label "D17" (at 85.09 90.17 0) (effects (font (size 1.27 1.27))))
+  (label "D14" (at 85.09 97.79 0) (effects (font (size 1.27 1.27))))
+  (label "D38" (at 85.09 113.03 0) (effects (font (size 1.27 1.27))))
+  (label "D33" (at 85.09 125.73 0) (effects (font (size 1.27 1.27))))
+  (label "D2" (at 220.98 31.75 0) (effects (font (size 1.27 1.27))))
+  (label "D3" (at 220.98 57.15 0) (effects (font (size 1.27 1.27))))
+  (label "D7" (at 220.98 82.55 0) (effects (font (size 1.27 1.27))))
+  (label "D12" (at 220.98 107.95 0) (effects (font (size 1.27 1.27))))
+  (label "D27" (at 220.98 133.35 0) (effects (font (size 1.27 1.27))))
+  (label "D31" (at 220.98 158.75 0) (effects (font (size 1.27 1.27))))
+  (label "D1" (at 107.95 185.42 0) (effects (font (size 1.27 1.27))))
+  (label "D4" (at 129.54 185.42 0) (effects (font (size 1.27 1.27))))
+  (label "D8" (at 148.59 185.42 0) (effects (font (size 1.27 1.27))))
+  (label "D32" (at 83.82 167.64 0) (effects (font (size 1.27 1.27))))
+  (label "D30" (at 107.95 167.64 0) (effects (font (size 1.27 1.27))))
+  (label "D26" (at 129.54 167.64 0) (effects (font (size 1.27 1.27))))
+  (label "D9" (at 148.59 167.64 0) (effects (font (size 1.27 1.27))))
+  (label "D23" (at 96.52 96.52 0) (effects (font (size 1.27 1.27))))
+  (label "D14" (at 146.05 96.52 0) (effects (font (size 1.27 1.27))))
+  (label "D38" (at 171.45 96.52 0) (effects (font (size 1.27 1.27))))
+  (label "D34" (at 194.31 96.52 0) (effects (font (size 1.27 1.27))))
+  (label "D22" (at 99.06 134.62 0) (effects (font (size 1.27 1.27))))
+  (label "D21" (at 99.06 137.16 0) (effects (font (size 1.27 1.27))))
+  (label "D20" (at 99.06 139.7 0) (effects (font (size 1.27 1.27))))
+  (label "D16" (at 99.06 142.24 0) (effects (font (size 1.27 1.27))))
+  (label "D37" (at 133.35 134.62 0) (effects (font (size 1.27 1.27))))
+  (label "D39" (at 133.35 137.16 0) (effects (font (size 1.27 1.27))))
+  (label "D40" (at 133.35 139.7 0) (effects (font (size 1.27 1.27))))
+  (label "D41" (at 133.35 142.24 0) (effects (font (size 1.27 1.27))))
+  (label "D33" (at 101.6 66.04 0) (effects (font (size 1.27 1.27))))
+  (label "D35" (at 101.6 68.58 0) (effects (font (size 1.27 1.27))))
+  (label "D36" (at 101.6 71.12 0) (effects (font (size 1.27 1.27))))
+  (label "D10" (at 101.6 73.66 0) (effects (font (size 1.27 1.27))))
+  (label "D28" (at 101.6 76.2 0) (effects (font (size 1.27 1.27))))
+  (label "D25" (at 101.6 78.74 0) (effects (font (size 1.27 1.27))))
+  (label "D24" (at 101.6 81.28 0) (effects (font (size 1.27 1.27))))
+  (label "D11" (at 101.6 83.82 0) (effects (font (size 1.27 1.27))))
+  (label "D5" (at 105.41 123.19 0) (effects (font (size 1.27 1.27))))
+  (label "D17" (at 129.54 123.19 0) (effects (font (size 1.27 1.27))))
+  (label "D15" (at 154.94 123.19 0) (effects (font (size 1.27 1.27))))
+  (label "D13" (at 180.34 123.19 0) (effects (font (size 1.27 1.27))))
+  (label "D29" (at 204.47 123.19 0) (effects (font (size 1.27 1.27))))
 )
