File: project/haptic-console-control-unit-perfboard.kicad_pcb (KiCad board)
At the start: 2 copper layers, 90 x 144 mm, 31 parts, among them J1 JST-XH-5, J2 JST-XH-5

Commit message: final
Parts:
- moved J_TEENSY_A 5.68 mm to (12.7, 58.4)
- moved J_TEENSY_B 5.68 mm to (12.7, 73.7)
Routing:
- net (no net): vias 1448 -> 1496
