File: project/haptic-console-control-unit-perfboard.kicad_pcb (KiCad board)
At the start: 2 copper layers, 90 x 144 mm, 36 parts, among them J1 JST-XH-5, J2 JST-XH-5

Commit message: update wiring guide
Parts:
- moved TP4 2.54 mm to (81.3, 25.4)
- moved TP5 2.54 mm to (81.3, 22.9)
