File: project/haptic-console-control-unit.kicad_pcb (KiCad board)
At the start: 2 copper layers, 300 x 200 mm, 30 parts, among them J1 JST-XH-5, J2 JST-XH-5, U1 Teensy 4.1

Commit message: make pcb more readable
Parts:
- moved CB1 92.7 mm to (19.5, 110.0)
- moved CB2 92.7 mm to (49.5, 110.0)
- moved CB3 92.7 mm to (79.5, 110.0)
- moved CB4 92.7 mm to (109.5, 110.0)
- moved CB5 92.7 mm to (139.5, 110.0)
- moved R5 87.9 mm to (144.4, 90.0)
- moved R1 87.9 mm to (24.4, 90.0)
- moved R2 87.9 mm to (54.4, 90.0)
- moved R3 87.9 mm to (84.4, 90.0)
- moved R4 87.9 mm to (114.4, 90.0)
- moved B1 70.8 mm to (162.5, 110.0)
- moved B2 70.8 mm to (187.5, 110.0)
- moved B3 70.8 mm to (212.5, 110.0)
- moved B4 70.8 mm to (237.5, 110.0)
- moved B5 70.8 mm to (162.5, 130.0)
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Connections:
- J1 pad 1: /D0 -> (no net)
- J1 pad 2: /D1 -> (no net)
- J1 pad 3: /D2 -> (no net)
- J1 pad 4: /D3 -> (no net)
- J1 pad 5: GND -> (no net)
- J2 pad 1: /D4 -> (no net)
- J2 pad 2: /D5 -> (no net)
- J2 pad 3: /D6 -> (no net)
- J2 pad 4: /D7 -> (no net)
- J2 pad 5: GND -> (no net)
Other:
- board text removed: "ICSP"

Commit message: more readable
Parts:
- S1, S2, S3, S4, S5, S6: value JST-XH-8 -> JST-XH-6; footprint Connector_JST:JST_XH_B8B-XH-A_1x08_P2.50mm_Vertical -> JST_XH_B6B-XH-A_1x06_P2.50mm_Vertical
Connections:
- S1 pad 2: +5V -> +3V3
- S1 pad 3: +3V3 -> +5V
- S2 pad 2: +5V -> +3V3
- S2 pad 3: +3V3 -> +5V
- S3 pad 2: +5V -> +3V3
- S3 pad 3: +3V3 -> +5V
- S4 pad 2: +5V -> +3V3
- S4 pad 3: +3V3 -> +5V
- S5 pad 2: +5V -> +3V3
- S5 pad 3: +3V3 -> +5V
- S6 pad 2: +5V -> +3V3
- S6 pad 3: +3V3 -> +5V

Commit message: final
Parts:
- R1, R12, R13, R2, R3, R4, R5: footprint Resistor_THT:R_Axial_DIN0207_L6.3mm_D2.5mm_P10.16mm_Horizontal -> R_0603_1608Metric
- moved S4 241.1 mm to (21.1, 47.5)
- moved S1 235.2 mm to (21.1, 35.5)
- moved S5 227.0 mm to (42.5, 47.5)
- moved S2 216.3 mm to (42.5, 35.5)
- moved B8 214.9 mm to (25.4, 95.5)
- moved S6 213.4 mm to (63.9, 47.5)
- moved R12 203.0 mm to (35.0, 56.0)
- moved S3 198.9 mm to (63.9, 35.5)
- moved R13 186.9 mm to (50.0, 56.0)
- moved B4 179.9 mm to (59.6, 83.5)
- moved B7 179.1 mm to (36.8, 95.5)
- moved B3 166.4 mm to (48.2, 83.5)
- moved B2 153.0 mm to (36.8, 83.5)
- moved B6 143.5 mm to (48.2, 95.5)
- moved B1 139.6 mm to (25.4, 83.5)
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- renumbered NP to NP1
Connections:
- J1 pad 1: (no net) -> /D0
- J1 pad 2: (no net) -> /D1
- J1 pad 3: (no net) -> /D2
- J1 pad 4: (no net) -> /D3
- J1 pad 5: (no net) -> GND
- J2 pad 1: (no net) -> /D4
- J2 pad 2: (no net) -> /D5
- J2 pad 3: (no net) -> /D6
- J2 pad 4: (no net) -> /D7
- J2 pad 5: (no net) -> GND
- U1 pad 1: (no net) -> GND
- U1 pad 10: (no net) -> /D8
- U1 pad 11: (no net) -> /D9
- U1 pad 12: (no net) -> /D10
- U1 pad 13: (no net) -> /D11
- U1 pad 14: (no net) -> /D12
- U1 pad 15: (no net) -> +3V3
- U1 pad 16: (no net) -> /D24
- U1 pad 17: (no net) -> /D25
- U1 pad 18: (no net) -> /D26
- U1 pad 19: (no net) -> /D27
- U1 pad 2: (no net) -> /D0
- U1 pad 20: (no net) -> /D28
- U1 pad 21: (no net) -> /D29
- U1 pad 22: (no net) -> /D30
- U1 pad 23: (no net) -> /D31
- U1 pad 24: (no net) -> /D32
- U1 pad 25: (no net) -> /D33
- U1 pad 26: (no net) -> /D34
- U1 pad 27: (no net) -> /D35
- U1 pad 28: (no net) -> /D36
- U1 pad 29: (no net) -> /D37
- U1 pad 3: (no net) -> /D1
- U1 pad 30: (no net) -> /D38
- U1 pad 31: (no net) -> /IRQ4
- U1 pad 32: (no net) -> /IRQ5
- U1 pad 33: (no net) -> /IRQ6
- U1 pad 34: (no net) -> GND
- U1 pad 35: (no net) -> /D13
- U1 pad 36: (no net) -> /D14
- U1 pad 37: (no net) -> /IRQ1
- U1 pad 38: (no net) -> /IRQ2
- U1 pad 39: (no net) -> /IRQ3
- U1 pad 4: (no net) -> /D2
- U1 pad 40: (no net) -> /SDA
- U1 pad 41: (no net) -> /SCL
- U1 pad 42: (no net) -> /D20
- U1 pad 43: (no net) -> /D21
- U1 pad 44: (no net) -> /D22
- U1 pad 45: (no net) -> /D23
- U1 pad 46: (no net) -> +3V3
- U1 pad 47: (no net) -> GND
- U1 pad 48: (no net) -> +5V
- U1 pad 5: (no net) -> /D3
- U1 pad 51: (no net) -> +3V3
- U1 pad 52: (no net) -> GND
- U1 pad 55: (no net) -> +5V
- U1 pad 58: (no net) -> GND
- U1 pad 59: (no net) -> GND
- U1 pad 6: (no net) -> /D4
- U1 pad 64: (no net) -> GND
- U1 pad 7: (no net) -> /D5
- U1 pad 8: (no net) -> /D6
- U1 pad 9: (no net) -> /D7
Routing:
- net GND: track 0.00 -> 408.6 mm
- net +3V3: track 0.00 -> 172.8 mm, vias 0 -> 2
- net /D35: track 0.00 -> 135.0 mm, vias 0 -> 2
- net /D5: track 0.00 -> 133.2 mm
- net /D33: track 0.00 -> 129.4 mm
- net /SDA: track 0.00 -> 128.8 mm, vias 0 -> 2
- net /SCL: track 0.00 -> 121.9 mm, vias 0 -> 1
- net /D34: track 0.00 -> 118.6 mm
- net +5V: track 0.00 -> 118.1 mm
- net /D6: track 0.00 -> 117.7 mm, vias 0 -> 2
- net /D4: track 0.00 -> 113.6 mm, vias 0 -> 2
- net /D23: track 0.00 -> 113.2 mm, vias 0 -> 2
- net /D7: track 0.00 -> 112.9 mm, vias 0 -> 1
- net /D32: track 0.00 -> 111.4 mm, vias 0 -> 1
- net /D36: track 0.00 -> 110.9 mm, vias 0 -> 1
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Other:
- board size 300 x 200 mm -> 88 x 131 mm
